File: recur_control/recur_control.kicad_pcb (KiCad board)
At the start: 2 copper layers, 100 x 100 mm, 41 parts, among them J1 AudioJack2_SwitchT, J2 AudioJack2_SwitchT, J3 AudioJack2_SwitchT, J4 AudioJack2_SwitchT, SW1 SW_Push, SW10 SW_Push, SW11 SW_Push, SW12 SW_Push, SW13 SW_Push, SW14 SW_Push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

Commit message: clikr circuit revision and start of code
Parts:
- added R1: 1k, Resistor_THT:R_Axial_DIN0207_L6.3mm_D2.5mm_P7.62mm_Horizontal, F.Cu at (203.1, 69.2)
- added R2: 1k, Resistor_THT:R_Axial_DIN0207_L6.3mm_D2.5mm_P7.62mm_Horizontal, F.Cu at (199.5, 69.2)
- added R3: 1k, Resistor_THT:R_Axial_DIN0207_L6.3mm_D2.5mm_P7.62mm_Horizontal, F.Cu at (199.7, 66.4)
- added R4: 1k, Resistor_THT:R_Axial_DIN0207_L6.3mm_D2.5mm_P7.62mm_Horizontal, F.Cu at (203.2, 66.4)
- J1, J2, J3, J4: value AudioJack2_SwitchT -> mono_jack_3.5mm
- RV1, RV2, RV3, RV4: value R_POT -> 10k_pot
- SW1, SW10, SW11, SW12, SW13, SW14, SW15, SW16, SW17, SW18, SW19, SW2, SW20, SW3, SW4, SW5, SW6, SW7, SW8, SW9: value SW_Push -> Push
Connections:
- D1 pad 2: analog_6 -> Net-(D1-Pad2)
- D2 pad 2: analog_7 -> Net-(D2-Pad2)
- D3 pad 2: analog_4 -> Net-(D3-Pad2)
- D4 pad 2: analog_5 -> Net-(D4-Pad2)
- D5 pad 1: analog_6 -> Net-(D1-Pad2)
- D6 pad 1: analog_7 -> Net-(D2-Pad2)
- D7 pad 1: analog_4 -> Net-(D3-Pad2)
- D8 pad 1: analog_5 -> Net-(D4-Pad2)
- J1 pad T: analog_6 -> Net-(D1-Pad2)
- J2 pad T: analog_7 -> Net-(D2-Pad2)
- J3 pad T: analog_4 -> Net-(D3-Pad2)
- J4 pad T: analog_5 -> Net-(D4-Pad2)
Routing:
- net Net-(D1-Pad2): track 0.00 -> 108.2 mm
- net analog_6: track 88.8 -> 4.14 mm
- net Net-(D3-Pad2): track 0.00 -> 80.0 mm
- net Net-(D2-Pad2): track 0.00 -> 79.9 mm
- net analog_7: track 74.4 -> 8.69 mm
- net analog_4: track 73.4 -> 8.00 mm
- net Net-(D4-Pad2): track 0.00 -> 52.9 mm
- net analog_5: track 51.0 -> 4.05 mm
- net GND: track 33.0 -> 65.7 mm
Other:
- board text added: "_^ 07"
- board text added: "c_l_i_k_r v0_2 cyberboy666"
- board text added: "underscores.shop"
- board text removed: "recur_control v0_1 cyberboy666"
