File: recur_control/recur_control.sch (KiCad schematic (older format))
At the start: 37 parts, among them J1 AudioJack2_SwitchT, J2 AudioJack2_SwitchT, J3 AudioJack2_SwitchT, J4 AudioJack2_SwitchT, SW1 SW_Push, SW10 SW_Push, SW11 SW_Push, SW12 SW_Push, SW13 SW_Push, SW14 SW_Push, SW15 SW_Push, SW16 SW_Push, SW17 SW_Push, SW18 SW_Push, SW19 SW_Push, SW2 SW_Push, SW20 SW_Push, SW3 SW_Push, SW4 SW_Push, SW5 SW_Push, SW6 SW_Push, SW7 SW_Push, SW8 SW_Push, SW9 SW_Push, U1 ProMicro

Commit message: clikr circuit revision and start of code
Parts:
- added R1, R2, R3, R4: 1k, Resistor_THT:R_Axial_DIN0207_L6.3mm_D2.5mm_P7.62mm_Horizontal, symbol Device:R
- J1, J2, J3, J4: value AudioJack2_SwitchT -> mono_jack_3.5mm
- RV1, RV2, RV3, RV4: value R_POT -> 10k_pot
- SW1, SW10, SW11, SW12, SW13, SW14, SW15, SW16, SW17, SW18, SW19, SW2, SW20, SW3, SW4, SW5, SW6, SW7, SW8, SW9: value SW_Push -> Push
Connections:
- net analog_4: now also R1.1; no longer D3.2 (A), D7.1 (K), J3.T
- net analog_5: now also R2.1; no longer D4.2 (A), D8.1 (K), J4.T
- net analog_6: now also R3.1; no longer D1.2 (A), D5.1 (K), J1.T
- net analog_7: now also R4.1; no longer D2.2 (A), D6.1 (K), J2.T
- new net: D3.2 (A), D7.1 (K), J3.T, R1.2
- new net: D4.2 (A), D8.1 (K), J4.T, R2.2
- new net: D1.2 (A), D5.1 (K), J1.T, R3.2
- new net: D2.2 (A), D6.1 (K), J2.T, R4.2
Other:
- moved on the sheet: D1, D2, D4, D5, D6, D8, J1, J2, J4
